File: Inverter.kicad_sch (KiCad schematic)
At the start: 76 parts, among them Q2 BSC022N04LSATMA1, Q3 BSC022N04LSATMA1, Q4 BSC022N04LSATMA1, Q5 BSC022N04LSATMA1, Q6 BSC022N04LSATMA1, Q7 BSC022N04LSATMA1, U4 TMC6140, U5 TSC2011, U6 TSC2011

Commit message: last commit
Parts:
- R14, R15, R16, R17, R24, R25: Part (none) -> AC0603FR-072R2L
- R18, R19, R20: Part (none) -> AC0603FR-0733KL
- R21, R22, R23, R35, R36, R6: Part (none) -> AC0603FR-073K9L
- R9: Part (none) -> AC0603FR-0710KL
Changed lines of the file:
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@@
+      (effects (font (size 1.27 1.27)) hide)
+    )
+    (property "Part" "AC0603FR-072R2L" (id 4) (at 228.092 64.262 0)
       (effects (font (size 1.27 1.27)) hide)
     )
@@
       (effects (font (size 1.27 1.27)) hide)
     )
+    (property "Part" "AC0603FR-072R2L" (id 4) (at 228.092 82.042 0)
+      (effects (font (size 1.27 1.27)) hide)
+    )
     (pin "1")
     (pin "2")
@@
       (effects (font (size 1.27 1.27)) hide)
     )
+    (property "Part" "AC0603FR-072R2L" (id 4) (at 206.502 82.042 0)
+      (effects (font (size 1.27 1.27)) hide)
+    )
     (pin "1")
     (pin "2")
@@
       (effects (font (size 1.27 1.27)) hide)
     )
+    (property "Part" "AC0603FR-072R2L" (id 4) (at 206.502 64.262 0)
+      (effects (font (size 1.27 1.27)) hide)
+    )
     (pin "1")
     (pin "2")
@@
       (effects (font (size 1.27 1.27)) hide)
     )
+    (property "Part" "AC0603FR-072R2L" (id 4) (at 186.182 64.262 0)
+      (effects (font (size 1.27 1.27)) hide)
+    )
     (pin "1")
     (pin "2")
@@
       (effects (font (size 1.27 1.27)) hide)
     )
+    (property "Part" "AC0603FR-072R2L" (id 4) (at 184.912 82.042 0)
+      (effects (font (size 1.27 1.27)) hide)
+    )
     (pin "1")
     (pin "2")
@@
       (effects (font (size 1.27 1.27)) hide)
     )
+    (property "Part" "AC0603FR-073K9L" (id 4) (at 228.346 111.76 0)
+      (effects (font (size 1.27 1.27)) hide)
+    )
     (pin "1")
     (pin "2")
@@
       (effects (font (size 1.27 1.27)) hide)
     )
+    (property "Part" "AC0603FR-0733KL" (id 4) (at 213.106 145.796 0)
+      (effects (font (size 1.27 1.27)) hide)
+    )
     (pin "1")
     (pin "2")
@@
     )
     (property "Datasheet" "~" (id 3) (at 227.076 130.81 0)
+      (effects (font (size 1.27 1.27)) hide)
+    )
+    (property "Part" "AC0603FR-073K9L" (id 4) (at 227.076 130.81 0)
       (effects (font (size 1.27 1.27)) hide)
     )
@@
     )
     (property "Datasheet" "~" (id 3) (at 214.122 125.73 0)
+      (effects (font (size 1.27 1.27)) hide)
+    )
+    (property "Part" "AC0603FR-0733KL" (id 4) (at 214.122 125.73 0)
       (effects (font (size 1.27 1.27)) hide)
     )
@@
       (effects (font (size 1.27 1.27)) hide)
     )
+    (property "Part" "AC0603FR-073K9L" (id 4) (at 241.046 125.73 0)
+      (effects (font (size 1.27 1.27)) hide)
+    )
     (pin "1")
     (pin "2")
@@
     )
     (property "Datasheet" "~" (id 3) (at 241.554 106.68 0)
+      (effects (font (size 1.27 1.27)) hide)
+    )
+    (property "Part" "AC0603FR-073K9L" (id 4) (at 241.554 106.68 0)
       (effects (font (size 1.27 1.27)) hide)
     )
@@
       (effects (font (size 1.524 1.524)))
     )
+    (property "Part" "AC0603FR-0710KL" (id 5) (at 41.91 162.56 0)
+      (effects (font (size 1.27 1.27)) hide)
+    )
     (pin "1")
     (pin "2")
@@
       (effects (font (size 1.27 1.27)) hide)
     )
+    (property "Part" "AC0603FR-073K9L" (id 4) (at 240.284 146.05 0)
+      (effects (font (size 1.27 1.27)) hide)
+    )
     (pin "1")
     (pin "2")
@@
       (effects (font (size 1.27 1.27)) hide)
     )
+    (property "Part" "AC0603FR-073K9L" (id 4) (at 227.076 151.13 0)
+      (effects (font (size 1.27 1.27)) hide)
+    )
     (pin "1")
     (pin "2")
@@
       (effects (font (size 1.27 1.27)) hide)
     )
+    (property "Part" "AC0603FR-0733KL" (id 4) (at 214.122 106.68 0)
+      (effects (font (size 1.27 1.27)) hide)
+    )
