File: progetto_motor_controller.kicad_sch (KiCad schematic)
At the start: 47 parts, among them J1 USB_B_Micro, J2 Conn_01x06, J3 Conn_01x04, J4 Screw_Terminal_01x03, J5 Conn_01x05, J6 Conn_02x10_Odd_Even, J7 Conn_01x02, J9 Conn_01x03, Q1 BSC022N04LSATMA1, U1 STM32F303RETx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

Commit message: before load switch
Parts:
- added D9: DESD32VS2SO, Package_TO_SOT_SMD:SOT-23, symbol MyLibrary_PMSM:DESD32VS2SO
- added U10: 74LVC3G17, Package_SO:VSSOP-8_2.3x2mm_P0.5mm, symbol 74xGxx:74LVC3G17
Connections:
- net +3V3: now also U10.8 (VCC), U10.8 (VCC), U10.8 (VCC)
- net CAN_H: now also D9.1 (K)
- net CAN_L: now also D9.2 (K)
- net ENC_A: now also U1.39 (PC8), U10.7; no longer C39.1, R31.1, R32.1, U1.37 (PC6)
- net ENC_B: now also U1.37 (PC6), U10.2; no longer C40.1, R30.1, R33.1, U1.38 (PC7)
- net ENC_I: now also U1.38 (PC7), U10.5; no longer C41.1, R29.1, R34.1, U1.39 (PC8)
- net GND: now also D9.3 (A), U10.4 (GND), U10.4 (GND), U10.4 (GND)
- new net ENC_A_5V: C39.1, R31.1, R32.1, U10.1
- new net ENC_B_5V: C40.1, R30.1, R33.1, U10.3
- new net ENC_I_5V: C41.1, R29.1, R34.1, U10.6
Other:
- moved on the sheet: H1, H2, H3, H4, J3, U2

Commit message: final
Parts:
- added R39: 120, Resistor_SMD:R_1210_3225Metric, symbol Device:R_Small
- added TP1, TP30, TP31, TP32, TP33: Testpoint, MyLibrary:TestPoint_1.0mm, symbol Connector:TestPoint
- C1: Part (none) -> CL10A475KQ8NNWC
- C2, C3, C4, C5, C6: Part (none) -> CL05B104KA5NNNC
- C42: footprint Capacitor_SMD:C_0402_1005Metric -> Capacitor_SMD:C_0603_1608Metric; Part (none) -> CL10B105KA8NNNC
- C43: Part (none) -> CL05B103KB5NNNC
- C7, C9: Part (none) -> CL05C100JB5NNNC CL05C120JB5NNNC
- D4: Part (none) -> 1N4148WS
- D9: Part (none) -> DESD32VS2SO-7
- Q1: value BSC022N04LSATMA1 -> DMG3402L-7; Part (none) -> DMG3402L-7
- U1: Part (none) -> STM32F303RETx --------
- U10: Part (none) -> 74LVC3G34DC,125
- U2: Part (none) -> SN65HVD253D
- U3: footprint Package_TO_SOT_SMD:SOT-363_SC-70-6 -> Package_TO_SOT_SMD:SOT-23-6; Part (none) -> CM1231-02SO
- Y1: Part (none) -> ABM8-16.000MHZ-10-1-U-T
Connections:
- net +5V: no longer J1.1 (VBUS)
- net CAN_H: now also R39.2, TP1.1
- net CAN_L: now also R39.1, TP30.1
- net DRV_STRONG: now also U1.25 (PC5)
- net ENC_A_5V: now also TP32.1
- net ENC_B_5V: now also TP33.1
- net ENC_I_5V: now also TP31.1
- net USB_CONN_D+: now also U3.4 (I/O2); no longer U3.3 (I/O2)
- net USB_CONN_D-: now also U3.3 (I/O2); no longer U3.1 (I/O1)
- net USB_D+: now also U3.6 (I/O1); no longer U3.4 (I/O2)
- net USB_D-: now also U3.1 (I/O1); no longer U3.6 (I/O1)
- new net 5V_USB: J1.1 (VBUS)
- no-connect marks 14 -> 13
Other:
- sheet Power ports: added 5V_VBUS; removed none
- moved on the sheet: C39, C40, C41, C8, D9, J1, J2, J3, J4, J5, R29, R30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

Commit message: last commit
Parts:
- C1: Part CL10A475KQ8NNWC -> CL10A475KP8NNNC
- C39, C40, C41, C8: Part (none) -> CL10A225KO8NNNC
- D1: value LED_Small -> LED_RED; Part (none) -> B1931URO-20D000114U1930
- D2: value LED_Small -> LED_GREEN; Part (none) -> B19Y1NG--20C000113U1930
- R1, R7, R8: Part (none) -> AC0603FR-0710KL
- R2, R29, R30, R31: Part (none) -> AC0603JR-071K5L
- R32, R33, R34: value 1k5 -> 0R
- R5: value 1k5 -> 820
Changed lines of the file:
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@@
       (effects (font (size 1.27 1.27)) hide)
     )
-    (property "Part" "CL10A475KQ8NNWC" (id 4) (at 64.135 86.995 0)
+    (property "Part" "CL10A475KP8NNNC" (id 4) (at 64.135 86.995 0)
       (effects (font (size 1.27 1.27)) hide)
     )
@@
     )
     (property "Datasheet" "~" (id 3) (at 91.44 186.69 0)
+      (effects (font (size 1.27 1.27)) hide)
+    )
+    (property "Part" "AC0603FR-0710KL" (id 4) (at 91.44 186.69 0)
       (effects (font (size 1.27 1.27)) hide)
     )
@@
       (effects (font (size 1.27 1.27)) hide)
     )
+    (property "Part" "AC0603FR-0710KL" (id 4) (at 246.38 107.95 0)
+      (effects (font (size 1.27 1.27)) hide)
+    )
     (pin "1")
     (pin "2")
@@
       (effects (font (size 1.27 1.27)) (justify left))
     )
-    (property "Value" "1k5" (id 1) (at 160.655 72.644 90)
+    (property "Value" "0R" (id 1) (at 160.655 72.644 90)
       (effects (font (size 1.27 1.27)) (justify left))
     )
@@
       (effects (font (size 1.27 1.27)) (justify left))
     )
-    (property "Value" "1k5" (id 1) (at 154.813 70.104 90)
+    (property "Value" "0R" (id 1) (at 154.813 70.104 90)
       (effects (font (size 1.27 1.27)) (justify left))
     )
@@
       (effects (font (size 1.27 1.27)) hide)
     )
+    (property "Part" "CL10A225KO8NNNC" (id 4) (at 147.32 77.216 0)
+      (effects (font (size 1.27 1.27)) hide)
+    )
     (pin "1")
     (pin "2")
@@
     )
     (property "Datasheet" "~" (id 3) (at 141.478 77.216 0)
+      (effects (font (size 1.27 1.27)) hide)
+    )
+    (property "Part" "CL10A225KO8NNNC" (id 4) (at 141.478 77.216 0)
       (effects (font (size 1.27 1.27)) hide)
     )
@@
       (effects (font (size 1.27 1.27)) hide)
     )
+    (property "Part" "CL10A225KO8NNNC" (id 4) (at 191.262 31.242 0)
+      (effects (font (size 1.27 1.27)) hide)
+    )
     (pin "1")
     (pin "2")
@@
       (effects (font (size 1.27 1.27)) hide)
     )
+    (property "Part" "AC0603JR-071K5L" (id 4) (at 135.128 62.992 0)
+      (effects (font (size 1.27 1.27)) hide)
+    )
     (pin "1")
     (pin "2")
@@
       (effects (font (size 1.27 1.27)) (justify right))
     )
-    (property "Value" "LED_Small" (id 1) (at 90.17 150.495 90)
+    (property "Value" "LED_GREEN" (id 1) (at 90.17 150.495 90)
       (effects (font (size 1.27 1.27)) (justify right))
     )
@@
     )
     (property "Datasheet" "~" (id 3) (at 93.98 147.955 90)
+      (effects (font (size 1.27 1.27)) hide)
+    )
+    (property "Part" "B19Y1NG--20C000113U1930" (id 4) (at 93.98 147.955 0)
       (effects (font (size 1.27 1.27)) hide)
     )
@@
       (effects (font (size 1.27 1.27)) hide)
     )
+    (property "Part" "AC0603JR-071K5L" (id 4) (at 138.684 62.992 0)
+      (effects (font (size 1.27 1.27)) hide)
+    )
     (pin "1")
     (pin "2")
@@
       (effects (font (size 1.27 1.27)) hide)
     )
+    (property "Part" "AC0603FR-0710KL" (id 4) (at 250.19 114.3 0)
+      (effects (font (size 1.27 1.27)) hide)
+    )
     (pin "1")
     (pin "2")
@@
     )
     (property "Datasheet" "~" (id 3) (at 152.908 77.216 0)
+      (effects (font (size 1.27 1.27)) hide)
+    )
+    (property "Part" "CL10A225KO8NNNC" (id 4) (at 152.908 77.216 0)
       (effects (font (size 1.27 1.27)) hide)
     )
@@
       (effects (font (size 1.27 1.27)) hide)
     )
+    (property "Part" "AC0603JR-071K5L" (id 4) (at 142.24 62.992 0)
+      (effects (font (size 1.27 1.27)) hide)
+    )
     (pin "1")
     (pin "2")
@@
       (effects (font (size 1.27 1.27)) (justify left))
     )
-    (property "Value" "1k5" (id 1) (at 95.4786 157.353 0)
+    (property "Value" "820" (id 1) (at 95.4786 157.353 0)
       (effects (font (size 1.27 1.27)) (justify left))
     )
@@
       (effects (font (size 1.27 1.27)) hide)
     )
+    (property "Part" "AC0603JR-071K5L" (id 4) (at 87.63 156.21 0)
+      (effects (font (size 1.27 1.27)) hide)
+    )
     (pin "1")
     (pin "2")
@@
       (effects (font (size 1.27 1.27)) (justify right))
     )
-    (property "Value" "LED_Small" (id 1) (at 80.01 150.495 90)
+    (property "Value" "LED_RED" (id 1) (at 80.01 150.495 90)
       (effects (font (size 1.27 1.27)) (justify right))
     )
@@
       (effects (font (size 1.27 1.27)) hide)
     )
+    (property "Part" "B1931URO-20D000114U1930" (id 4) (at 87.63 147.955 0)
+      (effects (font (size 1.27 1.27)) hide)
+    )
     (pin "1")
     (pin "2")
@@
       (effects (font (size 1.27 1.27)) (justify left))
     )
-    (property "Value" "1k5" (id 1) (at 149.225 67.564 90)
+    (property "Value" "0R" (id 1) (at 149.225 67.564 90)
       (effects (font (size 1.27 1.27)) (justify left))
     )
@@
     )
     (path "/f9eb455a-f9b0-4a40-aeb8-7fec771c76fc"
-      (reference "D1") (unit 1) (value "LED_Small") (footprint "LED_SMD:LED_0603_1608Metric")
+      (reference "D1") (unit 1) (value "LED_RED") (footprint "LED_SMD:LED_0603_1608Metric")
     )
     (path "/8003fc62-5cde-4dbd-8839-6a5adde8c547"
-      (reference "D2") (unit 1) (value "LED_Small") (footprint "LED_SMD:LED_0603_1608Metric")
+      (reference "D2") (unit 1) (value "LED_GREEN") (footprint "LED_SMD:LED_0603_1608Metric")
     )
     (path "/00000000-0000-0000-0000-000061cd02c2/e5396af2-22f9-4aa5-97de-37833e73eff4"
@@
     )
     (path "/cff15a6b-3072-4001-adf2-5e0270fc2d40"
-      (reference "R5") (unit 1) (value "1k5") (footprint "Resistor_SMD:R_0603_1608Metric")
+      (reference "R5") (unit 1) (value "820") (footprint "Resistor_SMD:R_0603_1608Metric")
     )
     (path "/00000000-0000-0000-0000-000061cd02c2/e1011013-62a3-47d2-9a4f-ee5ec3ce63cf"
@@
     )
     (path "/fb1a2199-6aa7-4068-a769-c48b56750efb"
-      (reference "R32") (unit 1) (value "1k5") (footprint "Resistor_SMD:R_0603_1608Metric")
+      (reference "R32") (unit 1) (value "0R") (footprint "Resistor_SMD:R_0603_1608Metric")
     )
     (path "/101598c1-b16c-4946-b3be-8fbfe5272d98"
-      (reference "R33") (unit 1) (value "1k5") (footprint "Resistor_SMD:R_0603_1608Metric")
+      (reference "R33") (unit 1) (value "0R") (footprint "Resistor_SMD:R_0603_1608Metric")
     )
     (path "/09b1566a-db6a-4d4a-9bb6-054e1256cf29"
-      (reference "R34") (unit 1) (value "1k5") (footprint "Resistor_SMD:R_0603_1608Metric")
+      (reference "R34") (unit 1) (value "0R") (footprint "Resistor_SMD:R_0603_1608Metric")
     )
     (path "/00000000-0000-0000-0000-000061cd02c2/8d502617-6466-460e-b2a8-3b6b91dc8a06"
